File: wonder_reader/wonder_reader.kicad_sch (KiCad schematic)
At the start: 117 parts, among them J1 USB_C_Receptacle_USB2.0, J2 Conn_01x04_Pin, J3 speaker_socket, J4 Conn_01x03_Pin, J6 prog, J7 vibrator, J8 ffc_solenoid, J9 TF-115, Q4 DMG1012T, SW1 SW_Reset, SW10 SW_keb, SW11 SW_keb, SW12 SW_keb, SW13 SW_keb, SW14 SW_keb, SW15 SW_keb, SW16 SW_keb, SW17 SW_keb, SW19 SW_Push_SPDT, SW2 SW_keb, SW3 SW_keb, SW4 SW_keb, SW5 SW_keb, SW6 SW_keb, SW7 SW_keb, SW8 SW_keb, SW9 SW_keb, U1 ESP32-S3-WROOM-1, U10 DRV8837C, U2 DRV8834RGER, U3 MAX98357AEWL_T, U4 BQ25895RTWR, U5 TLV62569DBV, U6 AH49EZ3-G1, U7 74HC595, U8 DRV8837C, U9 DRV8837C

Commit message: Completed new wonder reader pcb
Parts:
- removed C1: 1uf, Capacitor_SMD:C_0402_1005Metric, symbol Device:C_Small
- removed C2: 100nf, Capacitor_SMD:C_0402_1005Metric, symbol Device:C_Small
- removed C3: 22uf, Capacitor_SMD:C_0805_2012Metric, symbol Device:C_Small
- removed D1: LED, LED_SMD:LED_0201_0603Metric, symbol Device:LED
- removed D15, D16: 1N4148W, Diode_SMD:D_SOD-123, symbol Diode:1N4148W
- removed J2: Conn_01x04_Pin, Connector_JST:JST_PH_S4B-PH-K_1x04_P2.00mm_Horizontal, symbol Connector:Conn_01x04_Pin
- removed J7: vibrator, Connector_JST:JST_PH_S2B-PH-K_1x02_P2.00mm_Horizontal, symbol Connector_Generic:Conn_01x02
- removed J8: ffc_solenoid, Connector_FFC-FPC:Hirose_FH12-6S-0.5SH_1x06-1MP_P0.50mm_Horizontal, symbol Connector_Generic_MountingPin:Conn_01x06_MountingPin
- removed Q4: DMG1012T, Package_TO_SOT_SMD:SOT-523, symbol Transistor_FET:DMG1012T
- removed R1, R10, R12, R13, R22: 10k, Resistor_SMD:R_0603_1608Metric, symbol Device:R
- removed R24, R25: 24, Resistor_SMD:R_2512_6332Metric, symbol Device:R
- removed R9: 0.1, Resistor_SMD:R_1210_3225Metric, symbol Device:R
- removed SW1: SW_Reset, Button_Switch_SMD:SW_SPST_CK_RS282G05A3, symbol Switch:SW_Push
- removed SW19: SW_Push_SPDT, footprint:SW_XKB_DM1-16UC-1, symbol Switch:SW_Push_SPDT
- removed SW5, SW9: SW_keb, Button_Switch_Keyboard:SW_Cherry_MX_1.00u_PCB, symbol Switch:SW_Push
- removed TP3: P_3.3v, TestPoint:TestPoint_Pad_2.0x2.0mm, symbol Connector:TestPoint_Probe
- removed TP4: P_GND, TestPoint:TestPoint_Pad_2.0x2.0mm, symbol Connector:TestPoint_Probe
- removed U10: DRV8837C, Package_SON:WSON-8-1EP_2x2mm_P0.5mm_EP0.9x1.6mm, symbol Driver_Motor:DRV8837C
- removed U2: DRV8834RGER, footprint:DRV8834RGER, symbol DRV8834RGER:DRV8834RGER
- removed U3: MAX98357AEWL_T, footprint:BGA9N40P3X3_134X143X69N, symbol MAX98357AEWL_T:MAX98357AEWL_T
- removed U6: AH49EZ3-G1, Package_TO_SOT_THT:TO-92S, symbol Sensor_Magnetic:DRV5055A2xLPGxQ1
- removed U7: 74HC595, Package_SO:SOIC-16W_5.3x10.2mm_P1.27mm, symbol 74xx:74HC595
- added C26: 100uf, Capacitor_SMD:CP_Elec_6.3x5.4, symbol Device:C_Polarized
- added C27, C33, C34, C36: 100nf, Capacitor_SMD:C_0402_1005Metric, symbol Device:C_Small
- added C28, C37: 1uf, Capacitor_SMD:C_0402_1005Metric, symbol Device:C_Small
- added C29: 10nf, Capacitor_SMD:C_0402_1005Metric, symbol Device:C_Small
- added C30, C31, C32: 100pf, Capacitor_SMD:C_0402_1005Metric, symbol Device:C_Small
- added C35: 22uf, Capacitor_SMD:C_0805_2012Metric, symbol Device:C_Small
- added H5: screw_bottom1, MountingHole:MountingHole_5.3mm_M5, symbol Mechanical:MountingHole
- added H6: screw_bottom2, MountingHole:MountingHole_5.3mm_M5, symbol Mechanical:MountingHole
- added J2: ffc_solenoid, Connector_FFC-FPC:Hirose_FH12-6S-0.5SH_1x06-1MP_P0.50mm_Horizontal, symbol Connector_Generic_MountingPin:Conn_01x06_MountingPin
- added J5: motor_connection, Connector_PinHeader_1.27mm:PinHeader_1x06_P1.27mm_Vertical, symbol Connector:Conn_01x06_Socket
- added J8: vibrator, Connector_PinHeader_1.27mm:PinHeader_1x02_P1.27mm_Vertical, symbol Connector:Conn_01x02_Socket
- added SW5: motor_limit, footprint:SW_XKB_DM1-16UC-1, symbol Switch:SW_SPDT
- added SW9: onoffswitch, Library:G-Switch MK-12C02-G025, symbol Switch:SW_SPDT
- added U10: MAX98357AETE+T, footprint:21-0136I_T1633-4_MXM, symbol MAX98357AETE_T:MAX98357AETE+T
- added U12: STM32L031G6Ux, Package_DFN_QFN:QFN-28_4x4mm_P0.5mm, symbol MCU_ST_STM32L0:STM32L031G6Ux
- added U2, U6, U7: DRV8837C, Package_SON:WSON-8-1EP_2x2mm_P0.5mm_EP0.9x1.6mm, symbol Driver_Motor:DRV8837C
- added s_link1: stm_32stlink, Connector_PinHeader_2.00mm:PinHeader_1x04_P2.00mm_Vertical, symbol Connector:Conn_01x04_Socket
- added s_prog1: stm32_prog, Connector_PinHeader_2.00mm:PinHeader_1x05_P2.00mm_Vertical, symbol Connector:Conn_01x05_Socket
- C4: value 2.2uf -> 100nf; footprint Capacitor_SMD:C_0603_1608Metric -> Capacitor_SMD:C_0402_1005Metric; LCSC Part C57895 -> C1525
- C5: value 10uf -> 100nf; footprint Capacitor_SMD:C_0805_2012Metric -> Capacitor_SMD:C_0402_1005Metric; LCSC Part C15850 -> C1525
- C6: value 10nf -> 100nf; footprint Capacitor_SMD:C_0201_0603Metric -> Capacitor_SMD:C_0402_1005Metric; LCSC Part C285010 -> C1525
- H1, H2, H3, H4: footprint MountingHole:MountingHole_3.2mm_M3 -> MountingHole:MountingHole_2.2mm_M2
- J3: footprint Connector_JST:JST_PH_S2B-PH-K_1x02_P2.00mm_Horizontal -> Connector_JST:JST_GH_BM02B-GHS-TBT_1x02-1MP_P1.25mm_Vertical; symbol Connector:Conn_01x02_Socket -> Connector_Generic_MountingPin:Conn_01x02_MountingPin; LCSC Part (none) -> C161690
- J4: value Conn_01x03_Pin -> batt_conn; LCSC Part (none) -> C157929
- R2, R3: value 51k -> 24; footprint Resistor_SMD:R_0603_1608Metric -> Resistor_SMD:R_2512_6332Metric
- R5: value 1.5k -> 10k
- R6, R7, R8: value 0.1 -> 10k; footprint Resistor_SMD:R_1210_3225Metric -> Resistor_SMD:R_0603_1608Metric
- SW10, SW11, SW12, SW13, SW14, SW15, SW16, SW17, SW2, SW3, SW4, SW6, SW7, SW8: footprint Button_Switch_Keyboard:SW_Cherry_MX_1.00u_PCB -> Kailh:SW_Kailh_Choc_V1
- TP1, TP2: footprint TestPoint:TestPoint_Pad_2.0x2.0mm -> TestPoint:TestPoint_Pad_1.0x1.0mm
- TP5: value P_step_ena -> nsleep; footprint TestPoint:TestPoint_Pad_2.0x2.0mm -> TestPoint:TestPoint_Pad_1.0x1.0mm
- TP6: value P_sol1 -> nsleep; footprint TestPoint:TestPoint_Pad_2.0x2.0mm -> TestPoint:TestPoint_Pad_1.0x1.0mm
- U1: footprint Espressif:ESP32-S3-WROOM-1U -> Espressif:ESP32-S3-WROOM-1
- esp_prog1: renamed from J6; value prog -> esp32_prog; footprint Connector_PinSocket_2.54mm:PinSocket_1x06_P2.54mm_Horizontal -> Connector_PinHeader_2.00mm:PinHeader_1x06_P2.00mm_Vertical
Connections:
- net step is gone; now on net key_c2: U1.17 (GPIO9/TOUCH9/ADC1_CH8/FSPIHD/SUBSPIHD)
- net vref0 is gone; now on net limit: R4.2
- net +3.3V: now also C23.2, C5.1, R4.1, R6.1, R7.1, R8.1, esp_prog1.5 (Pin_5), C27.1, C28.2, C29.1, C30.1, C31.1, C32.1, C33.1, C35.2, C36.2, J5.3 (Pin_3), U12.1 (VDD), U12.17 (VDD), U12.5 (VDDA), U2.8 (VCC), U6.8 (VCC), U7.8 (VCC), s_link1.4 (Pin_4), s_prog1.4 (Pin_4); no longer C22.1, C4.1, C7.1, C8.1, D2.1 (K), esp_prog1.3 (Pin_3)
- net +5V: now also C21.1, C22.1, C6.1, C26.1, C34.1, U2.1 (VM), U6.1 (VM), U7.1 (VM); no longer C21.2, C23.2
- net +BATT: no longer C5.1, C6.1
- net Earth: now also C21.2, C4.1, C6.2, esp_prog1.2 (Pin_2), C26.2, C27.2, C28.1, C29.2, C30.2, C31.2, C32.2, C33.2, C34.2, C35.1, C36.1, C37.1, J5.4 (Pin_4), SW5.3 (C), U10.11 (GND), U10.15 (GND), U10.2 (GAIN_SLOT), U10.3 (GND), U12.16 (VSS), U12.28 (VSS), U2.4 (GND), U2.9 (GND), U6.4 (GND), U6.9 (GND), U7.4 (GND), U7.9 (GND), s_link1.1 (Pin_1), s_prog1.1 (Pin_1); no longer C21.1, C4.2, R2.2, R3.2, R5.1, R6.1, R7.1, R8.1, esp_prog1.6 (Pin_6)
- net bat+: now also SW9.3 (C); no longer U4.13 (BAT), U4.14 (BAT)
- net bclk: now also U10.16 (BCLK)
- net boot: now also esp_prog1.6 (Pin_6); no longer esp_prog1.2 (Pin_2)
- net din: now also U10.1 (DIN)
- net key_c1: now also U1.15 (GPIO3/TOUCH3/ADC1_CH2); no longer U1.24 (GPIO47/SPICLK_P/SUBSPICLK_P_DIFF)
- net key_c2: no longer U1.25 (GPIO48/SPICLK_N/SUBSPICLK_N_DIFF)
- net key_c3: now also U1.23 (GPIO21); no longer U1.16 (GPIO46)
- net key_c4: now also U1.31 (GPIO38/FSPIWP/SUBSPIWP); no longer U1.26 (GPIO45)
- net key_r1: now also U1.32 (MTCK/GPIO39/CLK_OUT3/SUBSPICS1); no longer U1.35 (MTMS/GPIO42)
- net key_r2: now also U1.33 (MTDO/GPIO40/CLK_OUT2); no longer U1.34 (MTDI/GPIO41/CLK_OUT1)
- net key_r3: now also U1.34 (MTDI/GPIO41/CLK_OUT1); no longer U1.33 (MTDO/GPIO40/CLK_OUT2)
- net key_r4: now also U1.35 (MTMS/GPIO42); no longer U1.32 (MTCK/GPIO39/CLK_OUT3/SUBSPICS1)
- net limit: now also C19.1, R5.1, U12.3 (PC15); no longer U1.31 (GPIO38/FSPIWP/SUBSPIWP)
- net lrclk: now also U10.14 (LRCLK)
- net rst: now also R6.2, C37.2; no longer C19.1
- net rx: now also esp_prog1.3 (Pin_3); no longer esp_prog1.4 (Pin_4)
- net scl: now also R8.2
- net sda: now also R7.2
- net tx: now also esp_prog1.4 (Pin_4); no longer esp_prog1.5 (Pin_5)
- net vibro: now also U9.6 (IN1)
- net bat_stat: now reaches U4.4 (STAT)
- net bat_stat: now also TP5.1
- net at J3.2 (Pin_2): now also U10.9 (OUTP)
- net at J3.1 (Pin_1): now also U10.10 (OUTN)
- net at R2.1: now also U6.2 (OUT1)
- net at U9.2 (OUT1): now also D2.1 (K), J8.1 (Pin_1)
- net at R3.1: now also U7.2 (OUT1)
- net at D2.2 (A): now also U9.3 (OUT2), J8.2 (Pin_2)
- net at U8.3 (OUT2): now also J2.4 (Pin_4)
- net sol2-: now reaches U8.5 (IN2)
- net sol2-: now also U12.12 (PA6)
- net sol2+: now reaches U8.6 (IN1)
- net sol2+: now also U12.11 (PA5)
- net at R23.2: now also J2.3 (Pin_3)
- net at R5.2: now also SW5.2 (B); no longer R4.1
- removed net Isol_oe: U1.23 (GPIO21), U8.7 (~{SLEEP}), U9.7 (~{SLEEP})
- net dir: no longer names the net of U1.12 (GPIO8/TOUCH8/ADC1_CH7/SUBSPICS1)
- net hall_eff renamed peri_sleep
- net peri_sleep: now also U9.7 (~{SLEEP})
- net sol_clk renamed usart2_rx
- net usart2_rx: now also U12.9 (PA3), s_prog1.2 (Pin_2)
- net sol_dat: no longer names the net of U1.8 (GPIO15/U0RTS/ADC2_CH4/XTAL_32K_P)
- net sol_latch: no longer names the net of U1.9 (GPIO16/U0CTS/ADC2_CH5/XTAL_32K_N)
- net sol_oe renamed nsleep
- net nsleep: now also U8.7 (~{SLEEP}), U12.2 (PC14), U2.7 (~{SLEEP}), U6.7 (~{SLEEP}), U7.7 (~{SLEEP}); no longer U1.11 (GPIO18/U1RXD/ADC2_CH7/CLK_OUT3)
- removed net stepper_ena: TP5.1, U1.15 (GPIO3/TOUCH3/ADC1_CH2)
- new net: C7.1, C8.1, U10.7 (VDD), U10.8 (VDD)
- new net: SW9.2 (B), U4.13 (BAT), U4.14 (BAT)
- new net: J5.1 (Pin_1), U2.3 (OUT2)
- new net: J5.2 (Pin_2), U2.2 (OUT1)
- new net: J2.6 (Pin_6), U7.3 (OUT2)
- new net: J2.1 (Pin_1), R2.2
- new net: J2.2 (Pin_2), U6.3 (OUT2)
- new net: J2.5 (Pin_5), R3.2
- new net motor+: U12.23 (PA15), U2.6 (IN1)
- new net motor-: U12.24 (PB3), U2.5 (IN2)
- new net quadA: J5.5 (Pin_5), U12.6 (PA0)
- new net quadB: J5.6 (Pin_6), U12.7 (PA1)
- new net sol1+: U12.25 (PB6), U6.6 (IN1)
- new net sol1-: U12.26 (PB7), U6.5 (IN2)
- new net sol3+: U12.14 (PB0), U7.6 (IN1)
- new net sol3-: U12.13 (PA7), U7.5 (IN2)
- new net swclk: U12.22 (PA14), s_link1.2 (Pin_2)
- new net swdio: U12.21 (PA13), s_link1.3 (Pin_3)
- new net u_boot0: U1.16 (GPIO46), U12.27 (BOOT0), s_prog1.5 (Pin_5)
- new net u_rst: C4.2, U1.26 (GPIO45), U12.4 (NRST)
- new net usart2_tx: U1.11 (GPIO18/U1RXD/ADC2_CH7/CLK_OUT3), U12.8 (PA2), s_prog1.3 (Pin_3)
- no-connect marks 19 -> 30
Other:
- note added: "+ Host/Device"
- note added: "Carriage System"
- note added: "STM32 microcontroller system memory boot mode.pdf STM32L031xx bootloader flashing is USART2 Bootloader active by boot0=1 nBoot1(bit)=1 (nBoot1 already 1 by default)"
- note added: "Switching"
- note added: "Wonder Reader"
- note added: "adv: - on/off control safety - decoupling - more pins - no need shift register - quadrature timer support"
- note added: "jtag can be freed because use usb jtag ESP32-S3 2.6.4"
- note added: "quadrature timer2"
- note added: "serial prog"
- note added: "stm32 prog and comm"
- note removed: "1/16 microstep"
- note removed: "Stepper"
- note removed: "jtag can be freed because usb jtag ESP32-S3 2.3.3"
- note removed: "solenoid control"
- note removed: "trip_cur = (xVREF/5*RISENSE)"
- moved on the sheet: C16, C17, C24, C25, C7, C8, C9, D2, H1, H2, H3, H4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

Commit message: Updated pcb to lower costs and rectify faults
Parts:
- removed C12: 10uf, Capacitor_SMD:C_0805_2012Metric, symbol Device:C_Small
- removed R14: 5.23k, Resistor_SMD:R_0603_1608Metric, symbol Device:R
- removed R15: 30.1k, Resistor_SMD:R_0603_1608Metric, symbol Device:R
- added C1: 4.7uf, Capacitor_SMD:C_0805_2012Metric, symbol Device:C_Small
- added R1, R9: 10k, Resistor_SMD:R_0603_1608Metric, symbol Device:R
- C11: footprint Capacitor_SMD:C_0402_1005Metric -> Capacitor_SMD:C_0603_1608Metric; LCSC Part C307434 -> C1622
- C15, C26: LCSC Part C90273 -> C1622
- C17: value 33uf -> 10uf; footprint Capacitor_SMD:CP_Elec_5x5.4 -> Capacitor_SMD:C_0805_2012Metric; LCSC Part C72507 -> C15850
- C28, C37: LCSC Part C29266 -> C52923
- C29: LCSC Part C1525 -> C15195
- C35: LCSC Part C5674 -> C45783
- D10, D11, D12, D13, D14, D17, D18, D2, D3, D4, D5, D6, D7, D8, D9: LCSC Part C2099 -> C81598
- L1, L2: LCSC Part C89016 -> C295335
- R11: LCSC Part (none) -> C8218
- R16: value 442k -> 270k; LCSC Part (none) -> C103491
- R17: LCSC Part (none) -> C25803
- R18, R19, R20, R21, R4, R5, R6, R7, R8: LCSC Part (none) -> C25804
- SW9: LCSC Part C778186 -> C963206
Connections:
- net Earth: now also C1.1, R1.1
- net at U4.22 (REGN): now also C1.2, R9.2
- net t_pin: no longer names the net of J4.1 (Pin_1)
- net t_pin: no longer U4.11 (TS)
- new net: R1.2, R9.1, U4.11 (TS)
- no-connect marks 30 -> 31
